File: PCB/Oil_furnace_control/RP2040_base.sch.kicad_sch (KiCad schematic)
At the start: 33 parts, among them J1 USB_B_Micro, J2 Conn_01x02, K1 FINDER-36.11, Q1 BC817, U1 NCP1117-3.3_SOT223, U2 W25Q128JVS, U3 RP2040, U4 LTV-817M, Y1 ABLS-12.000MHZ-B4-T

Commit message: no change
Parts:
- added D2, D3, D4, D5: 1N4448W, Diode_SMD:D_SOD-123, symbol Diode:1N4448W
- added K2, K3, K4, K5: FINDER-36.11, Relay_THT:Relay_SPDT_Finder_36.11, symbol Relay:FINDER-36.11
- added Q2, Q3, Q4, Q5: BC817, Package_TO_SOT_SMD:SOT-23, symbol Transistor_BJT:BC817
- added R10, R11, R12, R13, R14, R15, R8, R9: 1k, symbol Device:R
- added U5, U6, U7, U8: LTV-817M, Package_DIP:DIP-4_W10.16mm, symbol Isolator:LTV-817M
Connections:
- net in is gone; now on net GPIO2: R7.1
- net +5V: now also D2.1 (K), D3.1 (K), D4.1 (K), D5.1 (K), K2.A1, K3.A1, K4.A1, K5.A1, U5.4, U6.4, U7.4, U8.4
- net GND: now also Q2.2 (E), Q3.2 (E), Q4.2 (E), Q5.2 (E), U5.2, U6.2, U7.2, U8.2
- net GPIO13: now also R14.1
- net GPIO4: now also R8.1
- net GPIO5: now also R10.1
- net GPIO6: now also R12.1
- new net: R8.2, U5.1
- new net: R9.1, U5.3
- new net: D5.2 (A), K5.A2, Q5.3 (C)
- new net: D2.2 (A), K2.A2, Q2.3 (C)
- new net: D3.2 (A), K3.A2, Q3.3 (C)
- new net: R15.1, U8.3
- new net: Q5.1 (B), R15.2
- new net: D4.2 (A), K4.A2, Q4.3 (C)
- new net: R11.1, U6.3
- new net: Q3.1 (B), R11.2
- new net: R14.2, U8.1
- new net: R12.2, U7.1
- new net: R13.1, U7.3
- new net: Q4.1 (B), R13.2
- new net: Q2.1 (B), R9.2
- new net: R10.2, U6.1
Other:
- note added: "Additional fan relay"
- note added: "Electrovalve relay"
- note added: "Fan relay"
- note added: "Heater Relay"
- note added: "Ignition magneto relay"
- note removed: "Relay module"
- moved on the sheet: C10, C11, C12, C13, C14, C15, C16, C2, C3, C6, C7, C8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
